Commit message: modify N1_23dof

File: description/robots/N1/N1_23dof.urdf (robot description, URDF)
Before this commit: robot N1, 29 links, 28 joints
Links:
- removed link base_link
- added link pelvis, mass 3.18; collision cylinder length=0.135 radius=0.065; visual mesh filename=meshes/pelvis.STL
- link camera_link: geometry visual mesh filename=meshes/camera_link.STL
- link imu_link: geometry visual mesh filename=meshes/imu_link.STL
- link left_end_effector_link: geometry collision sphere radius=0.02751; visual mesh filename=meshes/left_end_effector_link.STL
- link left_foot_pitch_link: geometry collision mesh filename=meshes/left_foot_pitch_link.STL; visual mesh filename=meshes/left_foot_pitch_link.STL
- link left_foot_roll_link: geometry visual mesh filename=meshes/left_foot_roll_link.STL
- link left_hand_yaw_link: geometry collision cylinder length=0.12 radius=0.032; visual mesh filename=meshes/left_hand_yaw_link.STL
- link left_lower_arm_pitch_link: geometry visual mesh filename=meshes/left_lower_arm_pitch_link.STL
- link left_shank_pitch_link: geometry collision cylinder length=0.2 radius=0.04; visual mesh filename=meshes/left_shank_pitch_link.STL
- link left_thigh_pitch_link: geometry visual mesh filename=meshes/left_thigh_pitch_link.STL
- link left_thigh_roll_link: geometry collision cylinder length=0.12 radius=0.0415; visual mesh filename=meshes/left_thigh_roll_link.STL
- link left_thigh_yaw_link: geometry collision cylinder length=0.19 radius=0.06; visual mesh filename=meshes/left_thigh_yaw_link.STL
- link left_upper_arm_pitch_link: geometry visual mesh filename=meshes/left_upper_arm_pitch_link.STL
- link left_upper_arm_roll_link: geometry collision sphere radius=0.032; visual mesh filename=meshes/left_upper_arm_roll_link.STL
- link left_upper_arm_yaw_link: geometry collision cylinder length=0.12 radius=0.032; visual mesh filename=meshes/left_upper_arm_yaw_link.STL
- link right_end_effector_link: geometry collision sphere radius=0.02751; visual mesh filename=meshes/right_end_effector_link.STL
- link right_foot_pitch_link: geometry collision mesh filename=meshes/right_foot_pitch_link.STL; visual mesh filename=meshes/right_foot_pitch_link.STL
- link right_foot_roll_link: geometry visual mesh filename=meshes/right_foot_roll_link.STL
- link right_hand_yaw_link: geometry collision cylinder length=0.12 radius=0.032; visual mesh filename=meshes/right_hand_yaw_link.STL
- link right_lower_arm_pitch_link: geometry visual mesh filename=meshes/right_lower_arm_pitch_link.STL
- link right_shank_pitch_link: geometry collision cylinder length=0.2 radius=0.04; visual mesh filename=meshes/right_shank_pitch_link.STL
- link right_thigh_pitch_link: geometry visual mesh filename=meshes/right_thigh_pitch_link.STL
- link right_thigh_roll_link: geometry collision cylinder length=0.12 radius=0.0415; visual mesh filename=meshes/right_thigh_roll_link.STL
- link right_thigh_yaw_link: geometry collision cylinder length=0.19 radius=0.06; visual mesh filename=meshes/right_thigh_yaw_link.STL
- link right_upper_arm_pitch_link: geometry visual mesh filename=meshes/right_upper_arm_pitch_link.STL
- link right_upper_arm_roll_link: geometry collision sphere radius=0.032; visual mesh filename=meshes/right_upper_arm_roll_link.STL
- link right_upper_arm_yaw_link: geometry collision cylinder length=0.12 radius=0.032; visual mesh filename=meshes/right_upper_arm_yaw_link.STL
- link torso_link: geometry collision cylinder length=0.22 radius=0.1; collision sphere radius=0.08
- link waist_yaw_link: geometry collision cylinder length=0.055 radius=0.06; visual mesh filename=meshes/waist_yaw_link.STL
Joints:
- joint imu_joint: parent base_link -> pelvis
- joint left_hip_pitch_joint: parent base_link -> pelvis
- joint right_hip_pitch_joint: parent base_link -> pelvis
- joint waist_yaw_joint: parent base_link -> pelvis
