Commit message: modify h1_19dof urdf xml

File: description/robots/h1/h1.urdf (robot description, URDF)
Before this commit: robot h1_description, 25 links, 24 joints
Links:
- link left_ankle_link: geometry collision box size=0.28 0.03 0.024; visual mesh filename=meshes/left_ankle_link.dae
- link left_elbow_link: geometry collision cylinder length=0.09 radius=0.03; visual mesh filename=meshes/left_elbow_link.dae
- link left_hip_pitch_link: geometry collision cylinder length=0.2 radius=0.05; visual mesh filename=meshes/left_hip_pitch_link.dae
- link left_hip_roll_link: geometry collision cylinder length=0.01 radius=0.02; visual mesh filename=meshes/left_hip_roll_link.dae
- link left_hip_yaw_link: geometry collision cylinder length=0.02 radius=0.01; visual mesh filename=meshes/left_hip_yaw_link.dae
- link left_knee_link: geometry collision cylinder length=0.2 radius=0.05; visual mesh filename=meshes/left_knee_link.dae
- link left_shoulder_pitch_link: geometry collision cylinder length=0.04 radius=0.03; visual mesh filename=meshes/left_shoulder_pitch_link.dae
- link left_shoulder_roll_link: geometry collision cylinder length=0.01 radius=0.04; visual mesh filename=meshes/left_shoulder_roll_link.dae
- link left_shoulder_yaw_link: geometry collision cylinder length=0.01 radius=0.04; visual mesh filename=meshes/left_shoulder_yaw_link.dae
- link logo_link: geometry visual mesh filename=meshes/logo_link.dae
- link pelvis: geometry collision sphere radius=0.05; visual mesh filename=meshes/pelvis.dae
- link right_ankle_link: geometry collision box size=0.28 0.03 0.024; visual mesh filename=meshes/right_ankle_link.dae
- link right_elbow_link: geometry collision cylinder length=0.09 radius=0.03; visual mesh filename=meshes/right_elbow_link.dae
- link right_hip_pitch_link: geometry collision cylinder length=0.2 radius=0.05; visual mesh filename=meshes/right_hip_pitch_link.dae
- link right_hip_roll_link: geometry collision cylinder length=0.01 radius=0.02; visual mesh filename=meshes/right_hip_roll_link.dae
- link right_hip_yaw_link: geometry collision cylinder length=0.02 radius=0.01; visual mesh filename=meshes/right_hip_yaw_link.dae
- link right_knee_link: geometry collision cylinder length=0.2 radius=0.05; visual mesh filename=meshes/right_knee_link.dae
- link right_shoulder_pitch_link: geometry collision cylinder length=0.04 radius=0.03; visual mesh filename=meshes/right_shoulder_pitch_link.dae
- link right_shoulder_roll_link: geometry collision cylinder length=0.01 radius=0.04; visual mesh filename=meshes/right_shoulder_roll_link.dae
- link right_shoulder_yaw_link: geometry collision cylinder length=0.01 radius=0.04; visual mesh filename=meshes/right_shoulder_yaw_link.dae
- link torso_link: geometry collision box size=0.08 0.16 0.1; visual mesh filename=meshes/torso_link.dae

Commit message: finish train vision

File: description/robots/h1/h1.urdf (robot description, URDF)
Before this commit: robot h1_description, 25 links, 24 joints
Links:
- link left_ankle_link: geometry collision box size=0.28 0.03 0.024; visual mesh filename=meshes/left_ankle_link.STL
- link left_elbow_link: geometry collision cylinder length=0.09 radius=0.03; visual mesh filename=meshes/left_elbow_link.STL
- link left_hip_pitch_link: geometry collision cylinder length=0.2 radius=0.05; visual mesh filename=meshes/left_hip_pitch_link.STL
- link left_hip_roll_link: geometry collision cylinder length=0.01 radius=0.02; visual mesh filename=meshes/left_hip_roll_link.STL
- link left_hip_yaw_link: geometry collision cylinder length=0.02 radius=0.01; visual mesh filename=meshes/left_hip_yaw_link.STL
- link left_knee_link: geometry collision cylinder length=0.2 radius=0.05; visual mesh filename=meshes/left_knee_link.STL
- link left_shoulder_pitch_link: geometry collision cylinder length=0.04 radius=0.03; visual mesh filename=meshes/left_shoulder_pitch_link.STL
- link left_shoulder_roll_link: geometry collision cylinder length=0.01 radius=0.04; visual mesh filename=meshes/left_shoulder_roll_link.STL
- link left_shoulder_yaw_link: geometry collision cylinder length=0.01 radius=0.04; visual mesh filename=meshes/left_shoulder_yaw_link.STL
- link logo_link: geometry visual mesh filename=meshes/logo_link.STL
- link pelvis: geometry collision sphere radius=0.05; visual mesh filename=meshes/pelvis.STL
- link right_ankle_link: geometry collision box size=0.28 0.03 0.024; visual mesh filename=meshes/right_ankle_link.STL
- link right_elbow_link: geometry collision cylinder length=0.09 radius=0.03; visual mesh filename=meshes/right_elbow_link.STL
- link right_hip_pitch_link: geometry collision cylinder length=0.2 radius=0.05; visual mesh filename=meshes/right_hip_pitch_link.STL
- link right_hip_roll_link: geometry collision cylinder length=0.01 radius=0.02; visual mesh filename=meshes/right_hip_roll_link.STL
- link right_hip_yaw_link: geometry collision cylinder length=0.02 radius=0.01; visual mesh filename=meshes/right_hip_yaw_link.STL
- link right_knee_link: geometry collision cylinder length=0.2 radius=0.05; visual mesh filename=meshes/right_knee_link.STL
- link right_shoulder_pitch_link: geometry collision cylinder length=0.04 radius=0.03; visual mesh filename=meshes/right_shoulder_pitch_link.STL
- link right_shoulder_roll_link: geometry collision cylinder length=0.01 radius=0.04; visual mesh filename=meshes/right_shoulder_roll_link.STL
- link right_shoulder_yaw_link: geometry collision cylinder length=0.01 radius=0.04; visual mesh filename=meshes/right_shoulder_yaw_link.STL
- link torso_link: geometry collision box size=0.08 0.16 0.1; visual mesh filename=meshes/torso_link.STL
